Commit message: Add files via upload

File: ur5_robot.urdf.xacro (robot description, xacro)
@@ -17,9 +17,22 @@
     <origin xyz="0.0 0.0 0.72" rpy="2.35 0.0 3.14" />
   </joint>
-  <link name="probe"/>
+  <link name="probe">
+    <visual>
+      <origin xyz="-0.131 0 0" rpy="0 1.57 0"/>
+      <geometry>
+	<cylinder radius="0.10" length="0.262" />
+      </geometry>
+    </visual>
+    <collision>
+      <origin xyz="-0.131 0 0" rpy="0 1.57 0" />
+      <geometry>
+	<cylinder radius="0.10" length="0.262" />
+      </geometry>
+    </collision>
+  </link>
   <joint name="probe_joint" type="fixed">
     <parent link="ee_link" />
     <child link = "probe" />
-    <origin xyz="0.26 0.0 0.0" rpy="0.52359877559 0.0 0.0" />
+     <origin xyz="0.262 0.0 0.0" rpy="0.52359877559 0.0 0.0" />
   </joint>
 </robot>
